Commit message: modify limits of joints in urdf(xacro) after the official specification of irb140

File: abb_irb140_support/urdf/irb140.urdf (robot description, URDF)
Before this commit: robot abb_irb140, 9 links, 8 joints
Joints:
- joint joint_1: limit lower=-3.1416 upper=3.1416 effort=0 velocity=2.618 -> lower=-3.1416 upper=3.1416 effort=0 velocity=3.4907
- joint joint_2: limit lower=-1.7453 upper=1.9199 effort=0 velocity=2.618 -> lower=-1.5708 upper=1.9199 effort=0 velocity=3.4907; origin xyz=0.381 0.16 0.352 rpy=0 0 0 -> xyz=0.070 -0.041 0.352 rpy=0 0 0
- joint joint_3: limit lower=-1.0472 upper=1.1345 effort=0 velocity=2.618 -> lower=-4.0143 upper=0.8727 effort=0 velocity=4.5379
- joint joint_4: limit lower=-3.49 upper=3.49 effort=0 velocity=6.2832 -> lower=-2.8798 upper=2.8798 effort=0 velocity=6.2832
- joint joint_5: limit lower=-2.0944 upper=2.0944 effort=0 velocity=6.2832 -> lower=-2.0071 upper=2.0071 effort=0 velocity=6.2832
- joint joint_6: limit lower=-6.9813 upper=6.9813 effort=0 velocity=7.854 -> lower=-2.8449 upper=2.8449 effort=0 velocity=7.8540

File: abb_irb140_support/urdf/irb140_macro.xacro (robot description, xacro)
@@ -123,5 +123,5 @@
         <child link="${prefix}link_1"/>
         <axis xyz="0 0 1"/>
-        <limit lower="-3.1416" upper="3.1416" effort="0" velocity="2.618"/>
+        <limit lower="-3.1416" upper="3.1416" effort="0" velocity="3.4907"/>
     </joint>
     <joint name="${prefix}joint_2" type="revolute">
@@ -130,5 +130,5 @@
         <child link="${prefix}link_2"/>
         <axis xyz="0 1 0"/>
-        <limit lower="-1.7453" upper="1.9199" effort="0" velocity="2.618"/>
+        <limit lower="-1.5708" upper="1.9199" effort="0" velocity="3.4907"/>
     </joint>
     <joint name="${prefix}joint_3" type="revolute">
@@ -137,5 +137,5 @@
         <child link="${prefix}link_3"/>
         <axis xyz="0 1 0"/>
-        <limit lower="-1.0472" upper="1.1345" effort="0" velocity="2.618"/>
+        <limit lower="-4.0143" upper="0.8727" effort="0" velocity="4.5379"/>
     </joint>
     <joint name="${prefix}joint_4" type="revolute">
@@ -144,5 +144,5 @@
         <child link="${prefix}link_4"/>
         <axis xyz="1 0 0"/>
-        <limit lower="-3.49" upper="3.49" effort="0" velocity="6.2832"/>
+        <limit lower="-2.8798" upper="2.8798" effort="0" velocity="6.2832"/>
     </joint>
     <joint name="${prefix}joint_5" type="revolute">
@@ -151,5 +151,5 @@
         <child link="${prefix}link_5"/>
         <axis xyz="0 1 0"/>
-        <limit lower="-2.0944" upper="2.0944" effort="0" velocity="6.2832"/>
+        <limit lower="-2.0071" upper="2.0071" effort="0" velocity="6.2832"/>
     </joint>
     <joint name="${prefix}joint_6" type="revolute">
@@ -158,5 +158,5 @@
         <child link="${prefix}link_6"/>
         <axis xyz="1 0 0"/>
-        <limit lower="-6.9813" upper="6.9813" effort="0" velocity="7.854"/>
+        <limit lower="-2.8449" upper="2.8449" effort="0" velocity="7.8540"/>
     </joint>
     <joint name="${prefix}joint_6-tool0" type="fixed">
